File: bledevkitAC6329C4.kicad_sch (KiCad schematic)
At the start: 43 parts, among them J1 USB_C_Receptacle_USB2.0_16P, J2 Conn_01x02, J3 Conn_01x02, J4 Conn_01x07, J5 Qwiic_I2C_connector, J6 Conn_01x07, J7 Conn_01x01, J8 Conn_01x01, J9 Conn_01x02, SW1 SW_DPDT_x2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

Commit message: Initial BOM and Finalized graphics
Parts:
- AE1, JP1, JP4, JP5, TP1: now left out of the parts list
- D2: LCSC (none) -> C2856703
- D3: LCSC (none) -> C965790
- J2: LCSC (none) -> C7433648
- J3, J9, JP3, JP6: LCSC (none) -> C492401
- J4, J6: LCSC (none) -> C492406
- J7, J8: LCSC (none) -> C492400
- R6, R7: LCSC (none) -> C25123
- SW3: LCSC (none) -> C455280
- U3: LCSC (none) -> C3015484
- U4: value ATtiny202-SS -> ATtiny412-SSNR; LCSC (none) -> C1337190
Changed lines of the file:
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@@
 			)
 		)
+		(property "LCSC" "C492401"
+			(at 118.11 53.34 0)
+			(effects
+				(font
+					(size 1.27 1.27)
+				)
+				(hide yes)
+			)
+		)
 		(pin "2"
 		)
@@
 			)
 		)
+		(property "LCSC" "C492400"
+			(at 104.14 26.67 0)
+			(effects
+				(font
+					(size 1.27 1.27)
+				)
+				(hide yes)
+			)
+		)
 		(pin "1"
 		)
@@
 			)
 		)
+		(property "LCSC" "C2856703"
+			(at 80.01 175.26 0)
+			(effects
+				(font
+					(size 1.27 1.27)
+				)
+				(hide yes)
+			)
+		)
 		(pin "2"
 		)
@@
 		(unit 1)
 		(exclude_from_sim no)
-		(in_bom yes)
+		(in_bom no)
 		(on_board yes)
 		(dnp no)
@@
 		(unit 1)
 		(exclude_from_sim no)
-		(in_bom yes)
+		(in_bom no)
 		(on_board yes)
 		(dnp no)
@@
 			)
 		)
+		(property "LCSC" "C492400"
+			(at 123.19 58.42 0)
+			(effects
+				(font
+					(size 1.27 1.27)
+				)
+				(hide yes)
+			)
+		)
 		(pin "1"
 		)
@@
 			)
 		)
+		(property "LCSC" "C965790"
+			(at 95.25 76.2 0)
+			(effects
+				(font
+					(size 1.27 1.27)
+				)
+				(hide yes)
+			)
+		)
 		(pin "2"
 		)
@@
 		(unit 1)
 		(exclude_from_sim no)
-		(in_bom yes)
+		(in_bom no)
 		(on_board yes)
 		(dnp no)
@@
 			)
 		)
-		(property "LCSC" ""
+		(property "LCSC" "C25123"
 			(at 80.01 167.64 0)
 			(effects
@@
 			)
 		)
+		(property "LCSC" "C492406"
+			(at 226.06 144.78 0)
+			(effects
+				(font
+					(size 1.27 1.27)
+				)
+				(hide yes)
+			)
+		)
 		(pin "5"
 		)
@@
 			)
 		)
+		(property "LCSC" "C492406"
+			(at 255.27 144.78 0)
+			(effects
+				(font
+					(size 1.27 1.27)
+				)
+				(hide yes)
+			)
+		)
 		(pin "5"
 		)
@@
 			)
 		)
+		(property "LCSC" "C455280"
+			(at 83.82 161.29 0)
+			(effects
+				(font
+					(size 1.27 1.27)
+				)
+				(hide yes)
+			)
+		)
 		(pin "2"
 		)
@@
 			)
 		)
-		(property "LCSC" ""
+		(property "LCSC" "C25123"
 			(at 95.25 68.58 0)
 			(effects
@@
 		(unit 1)
 		(exclude_from_sim no)
-		(in_bom yes)
+		(in_bom no)
 		(on_board yes)
 		(dnp no)
@@
 			)
 		)
+		(property "LCSC" "C492401"
+			(at 106.68 109.22 0)
+			(effects
+				(font
+					(size 1.27 1.27)
+				)
+				(hide yes)
+			)
+		)
 		(pin "1"
 		)
@@
 			)
 		)
+		(property "LCSC" "C492401"
+			(at 57.15 109.22 0)
+			(effects
+				(font
+					(size 1.27 1.27)
+				)
+				(hide yes)
+			)
+		)
 		(pin "1"
 		)
@@
 			)
 		)
-		(property "Value" "ATtiny202-SS"
+		(property "Value" "ATtiny412-SSNR"
 			(at 36.83 167.6399 0)
 			(effects
@@
 			)
 		)
+		(property "LCSC" "C1337190"
+			(at 49.53 166.37 0)
+			(effects
+				(font
+					(size 1.27 1.27)
+				)
+				(hide yes)
+			)
+		)
 		(pin "2"
 		)
@@
 		(at 210.82 97.79 180)
 		(unit 1)
-		(exclude_from_sim yes)
+		(exclude_from_sim no)
 		(in_bom no)
 		(on_board yes)
@@
 		(mirror x)
 		(unit 1)
-		(exclude_from_sim yes)
+		(exclude_from_sim no)
 		(in_bom no)
 		(on_board yes)
@@
 			)
 		)
+		(property "LCSC" "C492401"
+			(at 99.06 21.59 0)
+			(effects
+				(font
+					(size 1.27 1.27)
+				)
+				(hide yes)
+			)
+		)
 		(pin "2"
 		)
@@
 			)
 		)
+		(property "LCSC" "C7433648"
+			(at 62.23 24.13 0)
+			(effects
+				(font
+					(size 1.27 1.27)
+				)
+				(hide yes)
+			)
+		)
 		(pin "2"
 		)
@@
 			)
 		)
+		(property "LCSC" "C3015484"
+			(at 118.11 72.39 0)
+			(effects
+				(font
+					(size 1.27 1.27)
+				)
+				(hide yes)
+			)
+		)
 		(pin "2"
 		)
@@
 		(unit 1)
 		(exclude_from_sim no)
-		(in_bom yes)
+		(in_bom no)
 		(on_board yes)
 		(dnp no)

Commit message: Started DFM optimization
Parts:
- C10, C5, C6, C8, C9: LCSC C14445 -> C52923
Connections:
- net EXT: now also SW2.3 (C); no longer SW2.4 (A)
- net VBUS: now also SW2.6 (C); no longer SW2.1 (A)
- net VSW: now also SW2.5 (B); no longer SW2.2 (B)
- net at JP6.1 (A): now also SW2.2 (B); no longer SW2.5 (B)
Other:
- moved on the sheet: SW2A, SW2B
Changed lines of the file:
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@@
 	(wire
 		(pts
+			(xy 73.66 55.88) (xy 73.66 50.8)
+		)
+		(stroke
+			(width 0)
+			(type default)
+		)
+	)
+	(wire
+		(pts
 			(xy 54.61 58.42) (xy 59.69 58.42)
 		)
@@
 	(wire
 		(pts
-			(xy 73.66 166.37) (xy 64.77 166.37)
+			(xy 77.47 21.59) (xy 77.47 24.13)
 		)
 		(stroke
@@
 	(wire
 		(pts
-			(xy 109.22 72.39) (xy 110.49 72.39)
+			(xy 73.66 166.37) (xy 64.77 166.37)
 		)
 		(stroke
@@
 	(wire
 		(pts
-			(xy 185.42 40.64) (xy 191.77 40.64)
+			(xy 109.22 72.39) (xy 110.49 72.39)
 		)
 		(stroke
@@
 	(wire
 		(pts
-			(xy 87.63 22.86) (xy 87.63 21.59)
+			(xy 185.42 40.64) (xy 191.77 40.64)
 		)
 		(stroke
@@
 	(wire
 		(pts
-			(xy 77.47 20.32) (xy 77.47 21.59)
-		)
-		(stroke
-			(width 0)
-			(type default)
-		)
-	)
-	(wire
-		(pts
 			(xy 215.9 105.41) (xy 215.9 107.95)
 		)
@@
 	(wire
 		(pts
-			(xy 64.77 50.8) (xy 76.2 50.8)
+			(xy 64.77 50.8) (xy 73.66 50.8)
 		)
 		(stroke
@@
 	(wire
 		(pts
+			(xy 76.2 55.88) (xy 73.66 55.88)
+		)
+		(stroke
+			(width 0)
+			(type default)
+		)
+	)
+	(wire
+		(pts
 			(xy 185.42 45.72) (xy 191.77 45.72)
 		)
@@
 	(symbol
 		(lib_id "Switch:SW_DPDT_x2")
-		(at 81.28 53.34 0)
+		(at 82.55 21.59 0)
 		(mirror y)
 		(unit 1)
@@
 		(dnp no)
 		(property "Reference" "SW2"
-			(at 81.28 44.45 0)
+			(at 82.55 13.462 0)
 			(effects
 				(font
@@
 		)
 		(property "Value" "SW_DPDT_x2"
-			(at 81.28 46.99 0)
+			(at 82.55 16.002 0)
 			(effects
 				(font
@@
 		)
 		(property "Footprint" "maxfootprints:DPDT-Slide_top"
-			(at 81.28 53.34 0)
+			(at 82.55 21.59 0)
 			(effects
 				(font
@@
 		)
 		(property "Datasheet" "~"
-			(at 81.28 53.34 0)
+			(at 82.55 21.59 0)
 			(effects
 				(font
@@
 		)
 		(property "Description" "Switch, dual pole double throw, separate symbols"
-			(at 81.28 53.34 0)
+			(at 82.55 21.59 0)
 			(effects
 				(font
@@
 		)
 		(property "LCSC" "C2837066"
-			(at 81.28 53.34 0)
+			(at 82.55 21.59 0)
 			(effects
 				(font
@@
 			)
 		)
-		(property "LCSC" "C14445"
+		(property "LCSC" "C52923"
 			(at 171.45 39.37 0)
 			(effects
@@
 	(symbol
 		(lib_id "Switch:SW_DPDT_x2")
-		(at 82.55 22.86 0)
+		(at 81.28 53.34 0)
 		(mirror y)
 		(unit 2)
@@
 		(dnp no)
 		(property "Reference" "SW2"
-			(at 82.55 13.97 0)
+			(at 81.28 44.45 0)
 			(effects
 				(font
@@
 		)
 		(property "Value" "SW_DPDT_x2"
-			(at 82.55 16.51 0)
+			(at 81.28 46.99 0)
 			(effects
 				(font
@@
 		)
 		(property "Footprint" "maxfootprints:DPDT-Slide_top"
-			(at 82.55 22.86 0)
+			(at 81.28 53.34 0)
 			(effects
 				(font
@@
 		)
 		(property "Datasheet" "~"
-			(at 82.55 22.86 0)
+			(at 81.28 53.34 0)
 			(effects
 				(font
@@
 		)
 		(property "Description" "Switch, dual pole double throw, separate symbols"
-			(at 82.55 22.86 0)
+			(at 81.28 53.34 0)
 			(effects
 				(font
@@
 		)
 		(property "LCSC" "C2837066"
-			(at 82.55 22.86 0)
+			(at 81.28 53.34 0)
 			(effects
 				(font
@@
 			)
 		)
-		(property "LCSC" "C14445"
+		(property "LCSC" "C52923"
 			(at 179.07 39.37 0)
 			(effects
@@
 			)
 		)
-		(property "LCSC" "C14445"
+		(property "LCSC" "C52923"
 			(at 163.83 39.37 0)
 			(effects
@@
 			)
 		)
-		(property "LCSC" "C14445"
+		(property "LCSC" "C52923"
 			(at 109.22 76.2 0)
 			(effects
@@
 			)
 		)
-		(property "LCSC" "C14445"
+		(property "LCSC" "C52923"
 			(at 127 76.2 0)
 			(effects
